File: Hardware/PCB/Corps/ProjetCorps.kicad_pcb (KiCad board)
At the start: 4 copper layers, 60 x 58 mm, 64 parts, among them J101 Conn_01x02, J102 Conn_01x03, J103 Conn_01x03, J104 Conn_01x15, J105 Conn_ST_STDC14, SW101 SW_SPDT, SW102 SW_SPST, SW201 SW_SPST, SW301 SW_SPST, SW401 SW_SPST, SW501 SW_SPST, SW601 SW_SPST, SW701 SW_SPST, SW801 SW_SPST, U101 STM32L412KBTx, U103 AZ1117-3.3, U104 173010542

Commit message: update pcb
Routing:
- net GND: vias 114 -> 116
- net +5V: vias 2 -> 4
Changed lines of the file:
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@@
 		(tags "LQFP QFP")
 		(property "Reference" "U101"
-			(at -4.35 5.7 360)
+			(at -4.35 5.7 0)
 			(layer "F.SilkS")
 			(effects
@@
 		)
 		(property "Value" "STM32L412KBTx"
-			(at 0 5.88 270)
+			(at 0 5.88 -90)
 			(layer "F.Fab")
 			(effects
@@
 		)
 		(fp_text user "${REFERENCE}"
-			(at 0 0 270)
+			(at 0 0 -90)
 			(layer "F.Fab")
 			(effects
@@
 		)
 		(property "Value" "100n"
-			(at 0 1.16 360)
+			(at 0 1.16 0)
 			(layer "F.Fab")
 			(effects
@@
 		)
 		(fp_text user "${REFERENCE}"
-			(at 0 0 360)
+			(at 0 0 0)
 			(layer "F.Fab")
 			(effects
@@
 		)
 		(property "Value" "1k"
-			(at 0 1.17 360)
+			(at 0 1.17 0)
 			(layer "F.Fab")
 			(effects
@@
 		)
 		(fp_text user "${REFERENCE}"
-			(at 0 0 360)
+			(at 0 0 0)
 			(layer "F.Fab")
 			(effects
@@
 		(tags "resistor")
 		(property "Reference" "R101"
-			(at -1.39 0.45 270)
+			(at -1.39 0.45 -90)
 			(layer "F.SilkS")
 			(effects
@@
 	)
 	(via
-		(at 141 62)
+		(at 140 62)
 		(size 0.8)
 		(drill 0.4)
@@
 	)
 	(via
+		(at 143 90)
+		(size 0.8)
+		(drill 0.4)
+		(layers "F.Cu" "B.Cu")
+		(free yes)
+		(net 2)
+	)
+	(via
 		(at 156 72)
 		(size 0.8)
@@
 	)
 	(via
+		(at 144 90)
+		(size 0.8)
+		(drill 0.4)
+		(layers "F.Cu" "B.Cu")
+		(free yes)
+		(net 2)
+	)
+	(via
 		(at 111 102)
 		(size 0.8)
@@
 	)
 	(via
+		(at 148 93)
+		(size 0.8)
+		(drill 0.4)
+		(layers "F.Cu" "B.Cu")
+		(free yes)
+		(net 4)
+	)
+	(via
 		(at 148.4 91.5)
 		(size 0.8)
@@
 		(net 4)
 	)
+	(via
+		(at 149 93)
+		(size 0.8)
+		(drill 0.4)
+		(layers "F.Cu" "B.Cu")
+		(free yes)
+		(net 4)
+	)
 	(segment
 		(start 122.5 88.95)
@@
 		(polygon
 			(pts
-				(xy 128.5 96.5) (xy 145 94.5) (xy 145 101.5) (xy 128.5 99.5)
+				(xy 128 94) (xy 145 94) (xy 145 103) (xy 128 103)
 			)
 		)
@@
 		(polygon
 			(pts
-				(xy 131.7 91.2) (xy 147.6 90.3) (xy 149.2 90.3) (xy 149.2 92.7) (xy 147.6 92.7) (xy 131.7 93.3)
+				(xy 131.7 91.2) (xy 147.6 90.3) (xy 150 90.3) (xy 150 94) (xy 131.7 94)
 			)
 		)
