File: Hardware/PCB/Tete/Projet_Animatronic.kicad_sch (KiCad schematic)
At the start: 24 parts, among them J1 Conn_01x06, J2 Conn_01x06, J3 Conn_01x06, J4 Conn_01x15, J5 Conn_01x04, J6 Conn_01x04, U8 PCA9685PW

Commit message: update head pcb
Parts:
- removed C1, C4: 10u, Capacitor_SMD:C_0603_1608Metric_Pad1.08x0.95mm_HandSolder, symbol Device:C_Small
- removed C2, C3: 100n, Capacitor_SMD:C_0603_1608Metric_Pad1.08x0.95mm_HandSolder, symbol Device:C_Small
- removed R1, R2: 115, Resistor_SMD:R_0603_1608Metric_Pad0.98x0.95mm_HandSolder, symbol Device:R
- added C101: 100n, Capacitor_SMD:C_0402_1005Metric, symbol Device:C_Small
- added C104, C105, C108, C109, C112, C113: 10u, Capacitor_SMD:C_0603_1608Metric, symbol Device:C_Small
- J102: renamed from J6; footprint Connector_PinHeader_2.54mm:PinHeader_1x04_P2.54mm_Vertical -> Connector_JST:JST_XH_B4B-XH-A_1x04_P2.50mm_Vertical
- J103: renamed from J5; footprint Connector_PinHeader_2.54mm:PinHeader_1x04_P2.54mm_Vertical -> Connector_JST:JST_XH_B4B-XH-A_1x04_P2.50mm_Vertical
- renumbered H1 to H101, H2 to H102, H3 to H103, H4 to H104, J4 to J101, J2 to J104, J1 to J105, J3 to J106, U8 to U101, U7 to U102, U5 to U103, U2 to U104, U3 to U105, U4 to U106, U6 to U107, U9 to U108
Connections:
- net +5V: now also C101.1
- net GND: now also U101.23 (~{OE}), U101.25 (EXTCLK), C101.2, C104.2, C105.2, C108.2, C109.2, C112.2, C113.2
- net I2C_SCL: now also U101.26 (SCL)
- net I2C_SDA: now also U101.27 (SDA)
- net 5V_3: now reaches J104.3 (Pin_3), U106.2 (VO)
- net 5V_3: now also C112.1
- net 5V_4: now reaches J104.4 (Pin_4), U105.2 (VO)
- net 5V_4: now also C105.1
- net 5V_5: now reaches J104.5 (Pin_5), U104.2 (VO)
- net 5V_5: now also C109.1
- net 5V_6: now reaches J104.6 (Pin_6), U103.2 (VO)
- net 5V_6: now also C113.1
- net 5V_1: now reaches J104.1 (Pin_1), U108.2 (VO)
- net 5V_1: now also C104.1
- net 5V_2: now reaches J104.2 (Pin_2), U107.2 (VO)
- net 5V_2: now also C108.1
- no-connect marks 12 -> 10
Other:
- moved on the sheet: J101, J102, J103, J104, J105, J106, U102, U103, U104, U105, U106, U107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
