File: Hardware/PCB/Body/ProjetCorps.kicad_pcb (KiCad board)
At the start: 4 copper layers, 60 x 58 mm, 64 parts, among them J101 Conn_01x02, J102 Conn_01x03, J103 Conn_01x03, J104 Conn_01x15, J105 Conn_ST_STDC14, SW101 SW_SPDT, SW102 SW_SPST, SW201 SW_SPST, SW301 SW_SPST, SW401 SW_SPST, SW501 SW_SPST, SW601 SW_SPST, SW701 SW_SPST, SW801 SW_SPST, U101 STM32L412KBTx, U103 AZ1117-3.3, U104 173010542

Commit message: correct mistake body pcb
Routing:
- net GND: vias 116 -> 112
- added copper zone on F.Cu, net +5V
